File: main_board/brushless_motor_controller.kicad_sch (KiCad schematic)
At the start: 15 parts, among them U1 ATA6561, U2 Teensy4.1_DEV-16771, U3 OKI-78SR-5_1.5-W36-C

Commit message: Added some stuff to the hard ware. Mostly where to put circuits on the schematic
Connections:
- net RXD1: now also U2.7 (RX2)
- net TXD1: now also U2.1 (TX1)
Other:
- moved on the sheet: C1, C2, C3, C4, C5, C6, C7, Conn1A, Conn1B, D1, R1, R2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
