File: board/BrushlessMocoBoard.kicad_sch (KiCad schematic)
At the start: 0 parts

Commit message: Made layout adjustments according to board review.
Other:
- sheet Half-Bridges & Current Sensing ports: added TEST_OPN_U, TEST_OPN_V, TEST_OPN_W, TEST_OPO_U, TEST_OPO_V, TEST_OPO_W, TEST_OPP_U, TEST_OPP_V, TEST_OPP_W; removed none
- sheet Interfaces ports: added TEST_OPN_U, TEST_OPN_V, TEST_OPN_W, TEST_OPO_U, TEST_OPO_V, TEST_OPO_W, TEST_OPP_U, TEST_OPP_V, TEST_OPP_W; removed none
